Commit message: minor updates to get working for franka

File: franka_description/urdfs/fr3.urdf (robot description, URDF)
Before this commit: robot fr3, 12 links, 11 joints
Joints:
- joint pen_holder_joint: origin xyz=0 0 0.107 rpy=0 0 0 -> xyz=0 0 0.107 rpy=0 0 0.0
- joint pen_joint: origin xyz=0.04 0.0 0.0 rpy=0 0 0 -> xyz=0.04 0.0 0.0 rpy=0 0 0.0
- joint pen_joint_to_tip: origin xyz=0.0 0.0 0.14 rpy=0 0 0 -> xyz=0.0 0.0 0.157 rpy=0.0 0.0 0.0
